File: din_power_atm90e26.sch (KiCad schematic (older format))
At the start: 62 parts, among them J1 CONN_01X06, J2 VBAT, J3 CONN_01X08, J4 CONN_02X18, J5 CONN_01X08, U1 MCP73831-2-OT, U2 AP7365-33YG-13, U3 AP7365-33YG-13, U4 Hi-Link_SMPS, U5 dc-dc

Commit message: Begin migration to relay drivers
Parts:
- removed R18, R19, R20, R21, R28, R29, R30, R31: 5.8R, Resistors_SMD:R_0603, symbol R
- C1, C2, C3, C4, C5, C6, C7, C8, C9: symbol C -> device:C
- D1: symbol D_Schottky -> device:D_Schottky
- D2: symbol LED -> device:LED
- F1: symbol Polyfuse -> device:Polyfuse
- G1: symbol LOGO -> whatnick:LOGO
- J1: symbol CONN_01X06 -> Connector_Generic:Conn_01x06
- J2: symbol CONN_01X02 -> Connector_Generic:Conn_01x02
- J3, J5: symbol CONN_01X08 -> Connector_Generic:Conn_01x08
- J4: symbol CONN_02X18 -> Connector_Generic:Conn_02x18_Counter_Clockwise
- L1: symbol Ferrite_Bead_Small -> device:Ferrite_Bead_Small
- LOGO_OSHW1: symbol Logo_Open_Hardware_Small -> graphic:Logo_Open_Hardware_Small
- R1, R10, R11, R12, R13, R14, R15, R16, R17, R2, R22, R23, R24, R25, R26, R27, R3, R32, R33, R4, R5, R6, R7, R8, R9: symbol R -> device:R
- RV1, RV2, RV3: symbol Varistor -> device:Varistor
- SYM1: symbol SYM_Flash_Small -> graphic:SYM_Flash_Small
- U1: symbol MCP73831-2-OT -> battery_management:MCP73831-2-OT
- U5: symbol dc-dc -> dc-dc1:dc-dc
Connections:
- wire segments 110 -> 122
Other:
- note added: "Optocoupler driver"
- note removed: "Option N-CT2"

Commit message: Updates links to new KiCAD libraries
Parts:
- added U6: ILQ74, symbol Isolator:ILQ74
- J4: symbol Connector_Generic:Conn_02x18_Counter_Clockwise -> Connector_Generic:Conn_02x18_Odd_Even
- U2: symbol AP7365-33YG-13 -> Regulator_Linear:L78L33_SOT89
- U3: symbol AP7365-33YG-13 -> Regulator_Linear:L78L05_SOT89
- U4: symbol Hi-Link_SMPS -> Converter_ACDC:HLK-PM01
- U5: symbol dc-dc1:dc-dc -> dc-dc:dc-dc
Connections:
- wire segments 122 -> 123

Commit message: Ripped out routing and added individual optos
Parts:
- removed C4, C9: 1uF, Capacitors_SMD:C_0603, symbol device:C
- removed D1: D_Schottky, Diodes_SMD:D_SOD-323F, symbol device:D_Schottky
- removed D2: LED, LEDs:LED_0603, symbol device:LED
- removed J2: VBAT, Connectors_JST:JST_SH_BM02B-SRSS-TB_02x1.00mm_Straight, symbol Connector_Generic:Conn_01x02
- removed R32: 2K, Resistors_SMD:R_0603, symbol device:R
- removed R33: 1K, Resistors_SMD:R_0603, symbol device:R
- removed U1: MCP73831-2-OT, TO_SOT_Packages_SMD:SOT-23-5, symbol battery_management:MCP73831-2-OT
- removed U6: ILQ74, symbol Isolator:ILQ74
- added J2: Conn_01x04, Connector_JST:JST_SH_BM04B-SRSS-TB_1x04-1MP_P1.00mm_Vertical, symbol Connector_Generic:Conn_01x04
- added R18: R, Resistor_SMD:R_0603_1608Metric, symbol device:R
- added U1, U6, U7, U8: LTV-356T, Package_SO:SO-4_4.4x3.6mm_P2.54mm, symbol Isolator:LTV-356T
- U2: value AP7365-33YG-13 -> L78L33_SOT89
- U3: value AP7365-33YG-13 -> L78L05_SOT89
Connections:
- net labels added: LED_H1, LED_H2, LED_H3, LED_H4, LED_L, RE1_H, RE1_L, RE2_H, RE2_L, RE3_H, RE3_L, RE4_H, RE4_L
- wire segments 123 -> 99
Other:
- note added: "Power Systems - dual 3.3v LDO"
- note removed: "Power Systems - Battery and 3.3V"

Commit message: Added routing for Opto-driver based PCB
Parts:
- U1, U6, U7, U8: manf# (none) -> LTV-356T
Changed lines of the file:
@@
 F 2 "Package_SO:SO-4_4.4x3.6mm_P2.54mm" H 2890 4155 50  0001 L CIN
 F 3 "http://optoelectronics.liteon.com/upload/download/DS70-2001-010/S_110_LTV-356T%2020140520.pdf" H 3090 4355 50  0001 L CNN
+F 4 "LTV-356T" H 3090 4355 50  0001 C CNN "manf#"
 	1    3090 4355
 	1    0    0    -1
@@
 F 2 "Package_SO:SO-4_4.4x3.6mm_P2.54mm" H 2890 4775 50  0001 L CIN
 F 3 "http://optoelectronics.liteon.com/upload/download/DS70-2001-010/S_110_LTV-356T%2020140520.pdf" H 3090 4975 50  0001 L CNN
+F 4 "LTV-356T" H 3090 4975 50  0001 C CNN "manf#"
 	1    3090 4975
 	1    0    0    -1
@@
 F 2 "Package_SO:SO-4_4.4x3.6mm_P2.54mm" H 2890 5370 50  0001 L CIN
 F 3 "http://optoelectronics.liteon.com/upload/download/DS70-2001-010/S_110_LTV-356T%2020140520.pdf" H 3090 5570 50  0001 L CNN
+F 4 "LTV-356T" H 3090 5570 50  0001 C CNN "manf#"
 	1    3090 5570
 	1    0    0    -1
@@
 F 2 "Package_SO:SO-4_4.4x3.6mm_P2.54mm" H 2890 5965 50  0001 L CIN
 F 3 "http://optoelectronics.liteon.com/upload/download/DS70-2001-010/S_110_LTV-356T%2020140520.pdf" H 3090 6165 50  0001 L CNN
+F 4 "LTV-356T" H 3090 6165 50  0001 C CNN "manf#"
 	1    3090 6165
 	1    0    0    -1
@@
 Text GLabel 3390 6065 2    50   Input ~ 0
 RE4_H
+Text GLabel 5900 5450 3    60   Output ~ 0
+GNDPWR
 $EndSCHEMATC

Commit message: Finalize BOM and Gerbers
Parts:
- R1: value 5.8R -> 2.4R; manf# CPF0603B5R76E1 -> ERJ-3RQF2R4V
- R10, R11, R2, R3, R4, R8, R9: value 5.8R -> 2.4R
- R18: value R -> 330R; manf# (none) -> 603-RC0201JR-7D330RL
- U4: manf# (none) -> HLK-PM01
Changed lines of the file:
@@
 P 1080 4545
 F 0 "R1" V 873 4545 50  0000 C CNN
-F 1 "5.8R" V 964 4545 50  0000 C CNN
+F 1 "2.4R" V 964 4545 50  0000 C CNN
 F 2 "Resistors_SMD:R_0603" V 1010 4545 50  0001 C CNN
 F 3 "" H 1080 4545 50  0001 C CNN
-F 4 "CPF0603B5R76E1" H 1080 4545 60  0001 C CNN "manf#"
+F 4 "ERJ-3RQF2R4V" H 1080 4545 60  0001 C CNN "manf#"
 	1    1080 4545
 	-1   0    0    1
@@
 P 1080 4945
 F 0 "R2" V 873 4945 50  0000 C CNN
-F 1 "5.8R" V 964 4945 50  0000 C CNN
+F 1 "2.4R" V 964 4945 50  0000 C CNN
 F 2 "Resistors_SMD:R_0603" V 1010 4945 50  0001 C CNN
 F 3 "" H 1080 4945 50  0001 C CNN
@@
 P 1930 4545
 F 0 "R8" V 1723 4545 50  0000 C CNN
-F 1 "5.8R" V 1814 4545 50  0000 C CNN
+F 1 "2.4R" V 1814 4545 50  0000 C CNN
 F 2 "Resistors_SMD:R_0603" V 1860 4545 50  0001 C CNN
 F 3 "" H 1930 4545 50  0001 C CNN
@@
 P 1930 4945
 F 0 "R9" V 1723 4945 50  0000 C CNN
-F 1 "5.8R" V 1814 4945 50  0000 C CNN
+F 1 "2.4R" V 1814 4945 50  0000 C CNN
 F 2 "Resistors_SMD:R_0603" V 1860 4945 50  0001 C CNN
 F 3 "" H 1930 4945 50  0001 C CNN
@@
 P 1080 5545
 F 0 "R3" V 873 5545 50  0000 C CNN
-F 1 "5.8R" V 964 5545 50  0000 C CNN
+F 1 "2.4R" V 964 5545 50  0000 C CNN
 F 2 "Resistors_SMD:R_0603" V 1010 5545 50  0001 C CNN
 F 3 "" H 1080 5545 50  0001 C CNN
@@
 P 1080 6045
 F 0 "R4" V 873 6045 50  0000 C CNN
-F 1 "5.8R" V 964 6045 50  0000 C CNN
+F 1 "2.4R" V 964 6045 50  0000 C CNN
 F 2 "Resistors_SMD:R_0603" V 1010 6045 50  0001 C CNN
 F 3 "" H 1080 6045 50  0001 C CNN
@@
 P 1930 5545
 F 0 "R10" V 1723 5545 50  0000 C CNN
-F 1 "5.8R" V 1814 5545 50  0000 C CNN
+F 1 "2.4R" V 1814 5545 50  0000 C CNN
 F 2 "Resistors_SMD:R_0603" V 1860 5545 50  0001 C CNN
 F 3 "" H 1930 5545 50  0001 C CNN
@@
 P 1930 5995
 F 0 "R11" V 1723 5995 50  0000 C CNN
-F 1 "5.8R" V 1814 5995 50  0000 C CNN
+F 1 "2.4R" V 1814 5995 50  0000 C CNN
 F 2 "Resistors_SMD:R_0603" V 1860 5995 50  0001 C CNN
 F 3 "" H 1930 5995 50  0001 C CNN
@@
 F 1 "Hi-Link_SMPS" H 5600 3141 60  0000 C CNN
 F 2 "hi-link_smps:HKLPM01" H 850 -700 60  0001 C CNN
-F 3 "" H 850 -700 60  0001 C CNN
-F 4 "50:$2.74" H 5600 2600 60  0001 C CNN "kicost:pricing"
+F 3 "http://www.hlktech.net/product_detail.php?ProId=54" H 850 -700 60  0001 C CNN
+F 4 "HLK-PM01" H 5600 2600 50  0001 C CNN "manf#"
+F 5 "50:$2.74" H 5600 2600 60  0001 C CNN "kicost:pricing"
 	1    5600 2600
 	1    0    0    -1
@@
 P 2775 6920
 F 0 "R18" H 2845 6966 50  0000 L CNN
-F 1 "R" H 2845 6875 50  0000 L CNN
+F 1 "330R" H 2845 6875 50  0000 L CNN
 F 2 "Resistor_SMD:R_0603_1608Metric" V 2705 6920 50  0001 C CNN
 F 3 "~" H 2775 6920 50  0001 C CNN
+F 4 "603-RC0201JR-7D330RL" H 2775 6920 50  0001 C CNN "manf#"
 	1    2775 6920
 	1    0    0    -1
